File: Hardware/projects/eCVT 507/eCVT 507.sch (EAGLE design)
At the start: 111 parts, among them IC1 IPB180N06S4-H1, IC2 IPB180N06S4-H1, J1 UJ2-MIBH-4-MSMT, Q1 16MHz 18pF, SW1 SW, U1 ATXMEGA128A4U-AU, U2 VNH5019ATR-E, U3 VNH5019ATR-E

Commit message: Added level shifters, xbee, other fixes
Parts:
- added C12: (no value), rcl:C-USC0805
- added R11: 1.7K, rcl:R-US_R0805
- added R12: 3.3K, rcl:R-US_R0805
- added U$20, U$21, U$22, U$23, U$24, U$27, U$29: NC, ME507:NC
- added U4, U5: MC14504BDR2G, MC14504BDR2G:MC14504BDR2G
- added XB1: XBEE, xbee:XBEE
- C10: value (none) -> 10pF
- C8: value 30pF -> 0.1uF
- C9: value 30pF -> 10pF
Connections:
- net RX renamed TEENSY_RX
- net TX renamed TEENSY_TX
- new net ENGINE_SPEED_3V3: U1.PD0, U4.AOUT
- new net N$39: R11.2, X4-2.1
- new net N$40: U$20.D, XB1.VREF
- new net N$41: U$21.D, XB1.!CTS!/DIO7
- new net N$42: U$22.D, XB1.ON/!SLEEP
- new net N$43: U$23.D, XB1.ASSOC/DIO5
- new net N$44: U$24.D, XB1.!RTS!/DIO6
- new net N$47: U$27.D, XB1.AD1/DIO1
- new net N$49: U5.MODE
- new net N$50: U$29.D, XB1.AD0/DIO0
- new net PENC_INA_3V3: U1.PE0, U4.EOUT
- new net PENC_INB_3V3: U1.PE1, U4.FOUT
- new net PMOT_INA_3V3: U1.PC0, U5.AOUT
- new net PMOT_INB_3V3: U1.PC1, U5.BOUT
- new net PMOT_PWM_3V3: U1.PC4, U5.COUT
- new net RWHEEL_SPEED_3V3: U1.PD1, U4.DOUT
- new net SENC_INA_3V3: U1.PE2, U4.BOUT
- new net SENC_INB_3V3: U1.PE3, U4.COUT
- new net SMOT_INA_3V3: U1.PC2, U5.DOUT
- new net SMOT_INB_3V3: U1.PC3, U5.EOUT
- new net SMOT_PWM_3V3: U1.PC5, U5.FOUT
- new net XBEE_RX: U1.PC6, XB1.DOUT
- new net XBEE_TX: U1.PC7, XB1.DIN/!CONFIG
- net +3V3: now also U4.VDD, U5.VDD, XB1.VCC
- net +5V: now also U4.VCC, U5.VCC
- net AVCC: now also C8.1
- net BRAKE_PRESSURE: now also R11.1, R12.2; no longer X4-2.1
- net ENGINE_SPEED: now also U4.AIN; no longer U1.PD0
- net GND: now also C12.2, R12.1, U4.VSS, U5.VSS, XB1.GND
- net MISO: now also XB1.DIO12
- net MOSI: now also XB1.DIO4
- net N$15: now also C11.1; no longer C10.1
- net N$20: now also XB1.RSSI/PWM/DIO10; no longer U1.PC6
- net N$21: now also XB1.!DTR!/SLEEP_RQ/DIO8; no longer U1.PC7
- net N$32: now also C12.1; no longer C11.1
- net PENC_INA: now also U4.EIN; no longer U1.PE0
- net PENC_INB: now also U4.FIN; no longer U1.PE1
- net PMOT_INA: now also U5.AIN; no longer U1.PC0
- net PMOT_INB: now also U5.BIN; no longer U1.PC1
- net PMOT_PWM: now also U5.CIN; no longer U1.PC4
- net RWHEEL_SPEED: now also U4.DIN; no longer U1.PD1
- net SCK: now also XB1.AD2/DIO2
- net SENC_INA: now also U4.BIN; no longer U1.PE2
- net SENC_INB: now also U4.CIN; no longer U1.PE3
- net SMOT_INA: now also U5.DIN; no longer U1.PC2
- net SMOT_INB: now also U5.EIN; no longer U1.PC3
- net SMOT_PWM: now also U5.FIN; no longer U1.PC5
- net SS: now also XB1.AD3/DIO3
- net XTAL1: now also C9.1; no longer C8.1
- net XTAL2: now also C10.1; no longer C9.1
Other:
- note added: "XMEGA RX connected to Xbee TX. XMEGA TX connected to Xbee RX."

Commit message: Updated wiring schematic
Parts:
- removed IC2: IPB180N06S4-H1, infineon:IPB180N06S4-H1
- removed U$14, U$15, U$8, U$9: NC, ME507:NC
- added R13, R14: 1K, rcl:R-US_R0805
- added R15: 10K, rcl:R-US_R0805
- added R16: 1.5K, rcl:R-US_R0805
- added U$25, U$31, U$33: NC, ME507:NC
- C10, C9: value 10pF -> 30pF
- R1: value 1K -> 1.7K
- R10: value 1.5K -> 3.3K
- R11: value 1.7K -> 3.3K
- R12: value 3.3K -> 1K
- R2, R3: value 1K -> 3.3K
- R4: value 10K -> 3.3K
- R5: value 1.5K -> 1K
- R8: value 1K -> 10K
- R9: value 10K -> 1.5K
Connections:
- net !RESET/PDI_CLK renamed RESET/PDI_CLK
- removed net N$15: C11.1, R4.2, R5.2
- removed net N$22: U$11.D, U1.PA7
- removed net N$24: U$13.D, U1.PB1
- removed net N$25: U$14.D, U1.PB2
- removed net N$27: IC1.D, U2.VCC
- removed net N$32: C12.1, R10.2, R9.2
- removed net N$35: IC2.G, U3.CP
- removed net N$36: IC2.D, U3.VCC
- removed net N$49: U5.MODE
- new net BRAKE_PRESSURE_3V3: U1.PB0
- new net DRIVER_CP: IC1.G, U2.CP, U3.CP
- new net DRIVER_VCC: IC1.D, U2.VCC, U3.VCC
- new net N$128: U$13.D, U1.PC1
- new net N$133: U$33.D, U3.CS_DIS
- new net N$45: U$25.D, U1.PD3
- new net N$46: U$31.D, U2.CS_DIS
- new net N$48: U$6.D, U1.PC0
- new net PMOT_CS: C11.1, R8.2, R9.2, U1.PB2
- new net SMOT_CS: C12.1, R15.2, R16.2, U1.PB3
- new net TEENSY_SS: U1.PD0
- new net XBEE_SS: U1.PD1
- net +12V: no longer IC2.S
- net +5V: now also R10.2, R11.2, R3.2, R4.2
- net BRAKE_PRESSURE: now also R1.1, R2.2; no longer R11.1, R12.2, U1.PA0
- net ENGINE_SPEED_3V3: now also U1.PE0; no longer U1.PD0
- net GND: now also R16.1, R2.1, R9.1, U4.MODE, U5.MODE; no longer R10.1, R12.1, R5.1
- net N$1: now also U1.PD2; no longer U1.PA1
- net N$10: now also R4.1, U2.ENA/DIAGA; no longer U$10.D, U1.PA6
- net N$11: now also XB1.!RESET; no longer U1.VCC_3
- net N$12: now also R6.2; no longer R2.2
- net N$13: now also R8.1; no longer R4.1
- net N$18: now also R3.1, U2.ENB/DIAGB; no longer IC1.G, U2.CP
- net N$19: now also R7.2; no longer R3.2
- net N$2: now also U$10.D, U1.PC4; no longer U$6.D, U1.PA2
- net N$23: now also U1.PD4; no longer U1.PB0
- net N$26: now also U$7.D, U1.PB1; no longer U$15.D, U1.PB3
- net N$28: now also R12.2; no longer R6.2
- net N$29: now also R13.2; no longer R7.2
- net N$3: now also U$11.D, U1.PC5; no longer U$7.D, U1.PA3
- net N$30: now also R14.2; no longer R8.2
- net N$31: now also R15.1; no longer R9.1
- net N$39: now also R1.2; no longer R11.2
- net N$4: now also R11.1, U3.ENA/DIAGA; no longer U$8.D, U1.PA4
- net N$5: now also R5.2; no longer R1.2
- net N$6: now also R10.1, U3.ENB/DIAGB; no longer U$9.D, U1.PA5
- net PENC_INA_3V3: now also U1.PA4; no longer U1.PE0
- net PENC_INB_3V3: now also U1.PA5; no longer U1.PE1
- net PMOT_INA: now also R5.1; no longer R1.1
- net PMOT_INA_3V3: now also U1.PA0; no longer U1.PC0
- net PMOT_INB: now also R6.1; no longer R2.1
- net PMOT_INB_3V3: now also U1.PA1; no longer U1.PC1
- net PMOT_PWM: now also R7.1; no longer R3.1
- net PMOT_PWM_3V3: now also U1.PE2; no longer U1.PC4
- net RWHEEL_SPEED_3V3: now also U1.PE1; no longer U1.PD1
- net SENC_INA_3V3: now also U1.PA6; no longer U1.PE2
- net SENC_INB_3V3: now also U1.PA7; no longer U1.PE3
- net SMOT_INA: now also R12.1; no longer R6.1
- net SMOT_INA_3V3: now also U1.PA2; no longer U1.PC2
- net SMOT_INB: now also R13.1; no longer R7.1
- net SMOT_INB_3V3: now also U1.PA3; no longer U1.PC3
- net SMOT_PWM: now also R14.1; no longer R8.1
- net SMOT_PWM_3V3: now also U1.PE3; no longer U1.PC5
- net SS: no longer U1.PD4
- net TEENSY_RX: now also U1.PC2; no longer U1.PD2
- net TEENSY_TX: now also U1.PC3; no longer U1.PD3
- net VCC: now also U1.VCC_3
