File: Hardware/December 2019 Edition/EAGLE/projects/DAQ and eCVT/DAQ and eCVT.brd (EAGLE design)
At the start: 86.4 x 138.4 mm, 20 parts, among them J1 10118193-0001LF, J2 TBL004-508-06BE-2GY, J3 TBL004-508-06BE-2GY, J4 TBL004-508-06BE-2GY, J5 TBL004-508-06BE-2GY, J6 TBL004-508-06BE-2GY, J7 TBL004-508-06BE-2GY, U1 AM26LS32ACDR, U2 CD40109BNSR

Commit message: Finished board layout, need to add mounting holes and writing
Parts:
- added R3, R4, R5, R6: (no value), rcl:0204/7
- J1: value 10118193-0001LF -> UJ2-MIBH2-4-SMT-TR; device Micro USB:FCI_10118193-0001LF -> Micro USB:CUI_UJ2-MIBH2-4-SMT-TR
- moved U2 77.6 mm to (31.8, 38.1)
- moved R1 64.8 mm to (25.4, 55.9), turned to 180 degrees
- moved R2 59.8 mm to (38.1, 55.9), turned to 0 degrees
- moved C1 6.35 mm to (29.2, 130.8)
- moved C2 6.35 mm to (34.3, 130.8)
- moved XB1 5.68 mm to (50.8, 124.5)
- moved CR1 5.24 mm to (29.2, 135.9), turned to 180 degrees
- moved J6 4.58 mm to (76.2, 74.9)
- moved J7 4.58 mm to (76.2, 109.2)
- moved J1 3.81 mm to (19.1, 137.2)
- moved J4 3.81 mm to (76.2, 3.81)
- moved J5 3.81 mm to (76.2, 38.1)
- moved U$57 2.54 mm to (3.81, 132.1)
- moved U$2 2.54 mm to (1.27, 72.4)
- moved U$58 2.54 mm to (3.81, 116.8)
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Connections:
- removed net N$1 (its old number): U$1.3V3
- removed net N$21 (its old number): U$2.3V3
- removed net N$42: J1.S1, J1.S2, J1.S3, J1.S4, J1.S5, J1.S6
- new net FBRAKE_PRESSURE_W/O_RES: J3.3_A, J3.3_B, R1.2
- new net N$40: J1.SH1, J1.SH2, J1.SH3, J1.SH4, J1.SH5
- new net RBRAKE_PRESSURE_W/O_RES: J3.4_A, J3.4_B, R3.1
- net +3V3: now also U$1.3V3, U$2.3V3, U2.2
- net BACKSHIFT_LED_12V: now also R6.2; no longer R2.2
- net BACKSHIFT_LED_12V_W/O_RES: now also R6.1; no longer R2.1
- net FBRAKE_PRESSURE: now also R1.1, R2.1, U$1.34/A15, U$2.34/A15; no longer J3.3_A, J3.3_B, U$1.33/A14, U$2.33/A14
- net GND: now also R2.2, R4.1
- net RBRAKE_PRESSURE: now also R3.2, R4.2, U$1.33/A14, U$2.33/A14; no longer J3.4_A, J3.4_B, U$1.34/A15, U$2.34/A15
- net UPSHIFT_LED_12V: now also R5.1; no longer R1.1
- net UPSHIFT_LED_12V_W/O_RES: now also R5.2; no longer R1.2
Routing:
- net +3V3: track 0.00 -> 276.0 mm, vias 0 -> 4
- net LOGGER_BUTTON: track 0.00 -> 154.1 mm, vias 0 -> 2
- net MARKER_BUTTON: track 0.00 -> 143.6 mm, vias 0 -> 2
- net +5V: track 0.00 -> 108.4 mm, vias 0 -> 2
- net FRWHEEL_SPEED: track 0.00 -> 92.9 mm, vias 0 -> 1
- net FLWHEEL_SPEED: track 0.00 -> 86.8 mm, vias 0 -> 1
- net LAUNCH_CONTROL_BUTTON: track 0.00 -> 84.9 mm, vias 0 -> 2
- net RWHEELS_SPEED: track 0.00 -> 84.0 mm
- net ECVT_SPARE_DAC1: track 0.00 -> 81.0 mm, vias 0 -> 2
- net +12V: track 0.00 -> 80.0 mm, vias 0 -> 1
- net ENGINE_SPEED: track 0.00 -> 77.9 mm
- net LOGGING_STATUS_LED: track 0.00 -> 74.8 mm
- net ECVT_SPARE_DAC0: track 0.00 -> 73.8 mm, vias 0 -> 1
- net BACKSHIFT_LED: track 0.00 -> 72.6 mm
- net P_ENC_A: track 0.00 -> 70.5 mm, vias 0 -> 4
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- added copper zone on layer 16, net +12V
- added copper zone on layer 1, net +3V3
- added copper zone on layer 16, net +3V3
- added copper zone on layer 1, net +5V
- added copper zone on layer 16, net +5V
- added copper zone on layer 1, net DAQ_ECVT_CS
- added copper zone on layer 1, net DAQ_ECVT_SCK
- added copper zone on layer 16, net FBRAKE_PRESSURE
- added copper zone on layer 1, net FLWHEEL_SPEED
- added copper zone on layer 1, net FRWHEEL_SPEED
- added copper zone on layer 16, net GND
- added copper zone on layer 16, net RBRAKE_PRESSURE
Other:
- board size 86.4 x 138.4 mm -> 88.9 x 139.7 mm

Commit message: December 2019 board finished
Parts:
- moved R1 12.7 mm to (38.1, 55.9)
- moved R3 12.7 mm to (38.1, 50.8)
- moved R2 12.7 mm to (50.8, 55.9)
- moved R4 12.7 mm to (50.8, 50.8)
- renumbered CR1 to VOLT_REG, J1 to USB, J2 to WHEEL_SPEED, J3 to BRAKE_PRESSURE, J4 to DAQ_BUTTONS_LEDS, J5 to ECVT_BUTTONS_LEDS, J6 to SPARE_ANALOG_PWM_I2C, J7 to SPARE_ANALOG_DAC, U$1 to DAQ, U$2 to ECVT, U$32 to MOTOR_DRIVER, U$57 to PENC, U$58 to SENC, U1 to DIFF_LINE_REC, U2 to LEVEL_SHIFT, XB1 to XBEE
Connections:
- net BACKSHIFT_LED renamed BKSHIFT_LED
- net BACKSHIFT_LED_12V renamed BKSHIFT_LED_12V
- net DAQ_SPARE_DAC0 renamed DAQ_SPARE_A21_DAC0
- net DAQ_SPARE_DAC1 renamed DAQ_SPARE_A22_DAC1
- net ECVT_SPARE_DAC0 renamed ECVT_SPARE_A21_DAC0
- net ECVT_SPARE_DAC1 renamed ECVT_SPARE_A22_DAC1
- net P_ENC_A renamed PENC_A
- net P_ENC_B renamed PENC_B
- net P_ENC_CHA renamed PENC_CHA
- net P_ENC_CHA/ renamed PENC_CHA/
- net P_ENC_CHB renamed PENC_CHB
- net P_ENC_CHB/ renamed PENC_CHB/
- net P_MOT_CS renamed PMOT_CS
- net P_MOT_INA renamed PMOT_INA
- net P_MOT_INB renamed PMOT_INB
- net P_MOT_PWM renamed PMOT_PWM
- net S_ENC_A renamed SENC_A
- net S_ENC_B renamed SENC_B
- net S_ENC_CHA renamed SENC_CHA
- net S_ENC_CHA/ renamed SENC_CHA/
- net S_ENC_CHB renamed SENC_CHB
- net S_ENC_CHB/ renamed SENC_CHB/
- net S_MOT_CS renamed SMOT_CS
- net S_MOT_INA renamed SMOT_INA
- net S_MOT_INB renamed SMOT_INB
- net S_MOT_PWM renamed SMOT_PWM
Routing:
- net RBRAKE_PRESSURE_W/O_RES: track 16.5 -> 29.2 mm
- net FBRAKE_PRESSURE_W/O_RES: track 16.5 -> 29.2 mm
- net FBRAKE_PRESSURE: track 64.2 -> 51.5 mm
- net RBRAKE_PRESSURE: track 67.8 -> 55.1 mm
- net BKSHIFT_LED: track 72.6 -> 74.4 mm
- net UPSHIFT_LED: track 61.8 -> 63.6 mm
- net +12V: track 80.0 -> 80.7 mm
Other:
- board text added: "+5V IN/OUT +12V OUT FBRAKE IN RBRAKE IN GND GND"
- board text added: "+5V IN/OUT ENGINE IN RWHEELS IN FLWHEEL IN FRWHEEL IN GND"
- board text added: "DESIGNED BY RAHUL GOYAL DEC 2019"
- board text added: "GND BKSHIFT LED OUT UPSHIFT LED OUT LCHCTRL BUT IN +12V OUT +5V IN/OUT"
- board text added: "GND DAQ A19 PWM SDA DAQ A18 PWM SCL DAQ A17 PWM DAQ A16 PWM +3V3 IN/OUT"
- board text added: "GND ECVT A22 DAC1 ECVT A21 DAC0 DAQ A22 DAC1 DAQ A21 DAC0 +3V3 IN/OUT"
- board text added: "GND LOG STATUS LED OUT MARKER BUTTON IN LOGGER BUTTON IN +12V OUT +5V IN/OUT"
- board text added: "SEE BOTTOM FOR PORT LABELS"
