File: Hardware/December 2019 Edition/EAGLE/projects/DAQ and eCVT/DAQ and eCVT.brd (EAGLE design)
At the start: 88.9 x 139.7 mm, 24 parts

Commit message: Minor formatting update
Connections:
- new net N$41: LEVEL_SHIFT.12
Changed lines of the file:
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@@
 <contactref element="ECVT" pad="28"/>
+</signal>
+<signal name="N$41">
+<contactref element="LEVEL_SHIFT" pad="12"/>
 </signal>
 </signals>
