File: Hardware/December 2019 Edition/EAGLE/projects/DAQ and eCVT/DAQ and eCVT.sch (EAGLE design)
At the start: 38 parts

Commit message: Progress
Parts:
- added J1: 10118193-0001LF, Micro USB:10118193-0001LF
- added U$28, U$29, U$30, U$31, U$33, U$34, U$35, U$47, U$48, U$49, U$50, U$51, U$52, U$53, U$54: NC, ME507:NC
- added U$32: POLOLU_DUAL_VNH5019, Pololo Dual VNH5019:POLOLU_DUAL_VNH5019
- added XB1: XBEE, Xbee:XBEE
- U$1, U$2: value BAJA_TEENSY_3.5 -> TEENSY_3.5; device Teensy:BAJA_TEENSY_3.5 -> Teensy:TEENSY_3.5
Connections:
- new net N$39: J1.D-, U$28.D
- new net N$40: J1.D+, U$29.D
- new net N$41: J1.ID, U$30.D
- new net N$42: J1.SHIELD, U$31.D
- new net N$43: U$34.D, XB1.!RESET
- new net N$44: U$32.VOUT, U$33.D
- new net N$45: U$35.D, XB1.ON/!SLEEP
- new net N$46: U$47.D, XB1.RSSI/PWM/DIO10
- new net N$47: U$48.D, XB1.!DTR!/SLEEP_RQ/DIO8
- new net N$48: U$49.D, XB1.!CTS!/DIO7
- new net N$49: U$50.D, XB1.!RTS!/DIO6
- new net N$50: U$51.D, XB1.ASSOC/DIO5
- new net N$51: U$52.D, XB1.AD1/DIO1
- new net N$52: U$53.D, XB1.AD0/DIO0
- new net N$53: U$54.D, XB1.VREF
- net +3V3: now also U$32.3V3, U$32.M1EN, U$32.M2EN, U$32.VDD, XB1.VCC
- net +5V: now also J1.VUSB, U$32.5V
- net DAQ_XBEE_CS: now also XB1.AD3/DIO3
- net DAQ_XBEE_MISO: now also XB1.DIO12
- net DAQ_XBEE_MOSI: now also XB1.DIO4
- net DAQ_XBEE_RX: now also XB1.DOUT
- net DAQ_XBEE_SCK: now also XB1.AD2/DIO2
- net DAQ_XBEE_TX: now also XB1.DIN/!CONFIG
- net GND: now also J1.GND, U$32.GND, U$32.GND1, U$32.GND2, U$32.GND3, XB1.GND
- net P_MOT_CS: now also U$32.M1CS
- net P_MOT_INA: now also U$32.M1INA
- net P_MOT_INB: now also U$32.M1INB
- net P_MOT_PWM: now also U$32.M1PWM
- net S_MOT_CS: now also U$32.M2CS
- net S_MOT_INA: now also U$32.M2INA
- net S_MOT_INB: now also U$32.M2INB
- net S_MOT_PWM: now also U$32.M2PWM

Commit message: Finished schematic? (except LED wiring)
Parts:
- added C1: 0.1uF, rcl:C-USC0805
- added C2: 10uF, rcl:C-USC0805
- added CR1: LD1117V33, Voltage Regulator 3.3V:LD1117V33
- added CR2: ST26C32ABDR, Quadruple Line Receiver:ST26C32ABDR
- added J2, J3, J4, J5, J6, J7: TBL004-508-06BE-2GY, Screwless Terminal 6-Pole:TBL004-508-06BE-2GY
- added U$55, U$56: NC, ME507:NC
- added U$57, U$58: SHF-105-01-X-D-TH, Male Header 2x5 0.05in:SHF-105-01-X-D-TH
- added U$59, U$60, U$61, U$62, U$63, U$64, U$65, U$66: NC, ME 507:NC
Connections:
- new net +12V: J3.2, J4.2, J5.2
- new net N$54: U$2.VIN, U$55.D
- new net N$55: U$1.VIN, U$56.D
- new net N$56: U$57.9, U$61.D
- new net N$59: U$57.10, U$62.D
- new net N$64: U$57.4, U$59.D
- new net N$65: U$57.1, U$60.D
- new net N$68: U$58.4, U$63.D
- new net N$69: U$58.10, U$64.D
- new net N$70: U$58.1, U$65.D
- new net N$71: U$58.9, U$66.D
- new net P_ENC_CHA: CR2.AIN2, U$57.6
- new net P_ENC_CHA/: CR2.AIN1, U$57.5
- new net P_ENC_CHB: CR2.BIN2, U$57.8
- new net P_ENC_CHB/: CR2.BIN1, U$57.7
- new net S_ENC_CHA: CR2.CIN2, U$58.6
- new net S_ENC_CHA/: CR2.CIN1, U$58.5
- new net S_ENC_CHB: CR2.DIN2, U$58.8
- new net S_ENC_CHB/: CR2.DIN1, U$58.7
- net +3V3: now also C2.1, CR1.OUTPUT, J6.1, J7.1
- net +5V: now also C1.1, CR1.INPUT, CR2.EN, CR2.VCC, J2.1, J3.1, J4.1, J5.1, U$57.2, U$58.2; no longer U$1.VIN, U$2.VIN
- net BACKSHIFT_LED: now also J5.5
- net DAQ_SPARE_A16_PWM: now also J6.2
- net DAQ_SPARE_A17_PWM: now also J6.3
- net DAQ_SPARE_A18_PWM_SCL: now also J6.4
- net DAQ_SPARE_A19_PWM_SDA: now also J6.5
- net DAQ_SPARE_DAC0: now also J7.2
- net DAQ_SPARE_DAC1: now also J7.3
- net ECVT_SPARE_DAC0: now also J7.4
- net ECVT_SPARE_DAC1: now also J7.5
- net ENGINE_SPEED: now also J2.2
- net FBRAKE_PRESSURE: now also J3.3
- net FLWHEEL_SPEED: now also J2.4
- net FRWHEEL_SPEED: now also J2.5
- net GND: now also C1.2, C2.2, CR1.GROUND, CR2.!, CR2.GND, J2.6, J3.5, J3.6, J4.6, J5.6, J6.6, J7.6, U$57.3, U$58.3
- net LAUNCH_CONTROL_BUTTON: now also J5.3
- net LOGGER_BUTTON: now also J4.3
- net LOGGING_STATUS_LED: now also J4.5
- net MARKER_BUTTON: now also J4.4
- net P_ENC_A: now also CR2.AOUT
- net P_ENC_B: now also CR2.BOUT
- net RBRAKE_PRESSURE: now also J3.4
- net RWHEELS_SPEED: now also J2.3
- net S_ENC_A: now also CR2.COUT
- net S_ENC_B: now also CR2.DOUT
- net UPSHIFT_LED: now also J5.4

Commit message: Finished schematic!
Parts:
- removed CR2: ST26C32ABDR, Quadruple Line Receiver:ST26C32ABDR
- added R1, R2: (no value), rcl:R-US_0204/7
- added U$67, U$68: NC, ME 507:NC
- added U1: AM26LS32ACDR, Quad. Diff. Line Receiver:AM26LS32ACDR
- added U2: CD40109BNSR, Quad. Level Shifter:CD40109BNSR
Connections:
- new net BACKSHIFT_LED_12V: J5.5, R2.2
- new net BACKSHIFT_LED_12V_W/O_RES: R2.1, U2.G
- new net LOGGING_STATUS_LED_12V: J4.5, U2.E
- new net N$58: U$67.D, U2.F
- new net N$60: U$68.D, U2.B
- new net UPSHIFT_LED_12V: J5.4, R1.1
- new net UPSHIFT_LED_12V_W/O_RES: R1.2, U2.H
- net +12V: now also U2.VDD
- net +3V3: now also U2.ENABLEC, U2.ENABLED, U2.VCC
- net +5V: now also U1.G, U1.VCC; no longer CR2.EN, CR2.VCC
- net BACKSHIFT_LED: now also U2.C; no longer J5.5
- net GND: now also U1.!G, U1.GND, U2.ENABLEB, U2.VSS; no longer CR2.!, CR2.GND
- net LOGGING_STATUS_LED: now also U2.A; no longer J4.5
- net P_ENC_A: now also U1.1Y; no longer CR2.AOUT
- net P_ENC_B: now also U1.2Y; no longer CR2.BOUT
- net P_ENC_CHA: now also U1.1A; no longer CR2.AIN2
- net P_ENC_CHA/: now also U1.1B; no longer CR2.AIN1
- net P_ENC_CHB: now also U1.2A; no longer CR2.BIN2
- net P_ENC_CHB/: now also U1.2B; no longer CR2.BIN1
- net S_ENC_A: now also U1.3Y; no longer CR2.COUT
- net S_ENC_B: now also U1.4Y; no longer CR2.DOUT
- net S_ENC_CHA: now also U1.3A; no longer CR2.CIN2
- net S_ENC_CHA/: now also U1.3B; no longer CR2.CIN1
- net S_ENC_CHB: now also U1.4A; no longer CR2.DIN2
- net S_ENC_CHB/: now also U1.4B; no longer CR2.DIN1
- net UPSHIFT_LED: now also U2.D; no longer J5.4
Other:
- moved on the sheet: J2, J3, J4, J5, J6, J7, U$58

Commit message: Started board
Parts:
- removed U$33: NC, ME507:NC
Connections:
- removed net N$44: U$32.VOUT, U$33.D
- net +12V: now also U$32.VOUT
Changed lines of the file:
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@@
 <part name="FRAME1" library="ME507" deviceset="TITLEBLOCK_LET_L" device=""/>
 <part name="FRAME2" library="ME507" deviceset="TITLEBLOCK_LET_L" device=""/>
-<part name="J1" library="Micro USB" deviceset="10118193-0001LF" device=""/>
 <part name="U$28" library="ME507" deviceset="NC" device=""/>
 <part name="P+2" library="supply1" library_urn="urn:adsk.eagle:library:371" deviceset="+5V" device=""/>
@@
 <part name="U$2" library="Teensy" deviceset="TEENSY_3.5" device=""/>
 <part name="GND9" library="supply1" library_urn="urn:adsk.eagle:library:371" deviceset="GND" device=""/>
-<part name="U$33" library="ME507" deviceset="NC" device=""/>
 <part name="GND10" library="supply1" library_urn="urn:adsk.eagle:library:371" deviceset="GND" device=""/>
 <part name="+3V6" library="supply1" library_urn="urn:adsk.eagle:library:371" deviceset="+3V3" device=""/>
@@
 <part name="R1" library="rcl" library_urn="urn:adsk.eagle:library:334" deviceset="R-US_" device="0204/7" package3d_urn="urn:adsk.eagle:package:23498/2"/>
 <part name="R2" library="rcl" library_urn="urn:adsk.eagle:library:334" deviceset="R-US_" device="0204/7" package3d_urn="urn:adsk.eagle:package:23498/2"/>
+<part name="J1" library="Micro USB" deviceset="10118193-0001LF" device=""/>
+<part name="P+15" library="supply1" library_urn="urn:adsk.eagle:library:371" deviceset="+12V" device=""/>
 </parts>
 <sheets>
@@
 <attribute name="DRAWING_NAME" x="240.665" y="3.81" size="2.54" layer="94" align="bottom-right"/>
 </instance>
-<instance part="J1" gate="G$1" x="68.58" y="149.86" smashed="yes">
-<attribute name="NAME" x="63.49835" y="160.7886" size="1.778" layer="95"/>
-<attribute name="VALUE" x="63.49806875" y="137.1503" size="1.778" layer="96"/>
-</instance>
 <instance part="U$28" gate="A" x="58.42" y="154.94" smashed="yes" rot="R180"/>
 <instance part="P+2" gate="1" x="50.8" y="162.56" smashed="yes">
@@
 <attribute name="VALUE" x="96.52" y="58.42" size="1.778" layer="96"/>
 </instance>
-<instance part="U$33" gate="A" x="58.42" y="93.98" smashed="yes" rot="R180"/>
 <instance part="GND10" gate="1" x="53.34" y="101.6" smashed="yes" rot="R180">
 <attribute name="VALUE" x="55.88" y="104.14" size="1.778" layer="96" rot="R180"/>
@@
 <attribute name="VALUE" x="223.52" y="129.54" size="1.778" layer="96"/>
 </instance>
+<instance part="J1" gate="G$1" x="68.58" y="149.86" smashed="yes">
+<attribute name="NAME" x="63.49835" y="160.7886" size="1.778" layer="95"/>
+<attribute name="VALUE" x="63.49806875" y="137.1503" size="1.778" layer="96"/>
+</instance>
+<instance part="P+15" gate="1" x="48.26" y="101.6" smashed="yes">
+<attribute name="VALUE" x="45.72" y="96.52" size="1.778" layer="96" rot="R90"/>
+</instance>
 </instances>
 <busses>
 </busses>
 <nets>
-<net name="N$39" class="0">
-<segment>
-<pinref part="J1" gate="G$1" pin="D-"/>
-<pinref part="U$28" gate="A" pin="D"/>
-</segment>
-</net>
-<net name="N$40" class="0">
-<segment>
-<pinref part="U$29" gate="A" pin="D"/>
-<pinref part="J1" gate="G$1" pin="D+"/>
-</segment>
-</net>
-<net name="N$41" class="0">
-<segment>
-<pinref part="U$30" gate="A" pin="D"/>
-<pinref part="J1" gate="G$1" pin="ID"/>
-</segment>
-</net>
 <net name="+5V" class="0">
 <segment>
-<pinref part="J1" gate="G$1" pin="VUSB"/>
 <pinref part="P+2" gate="1" pin="+5V"/>
 <wire x1="58.42" y1="157.48" x2="50.8" y2="157.48" width="0.1524" layer="91"/>
 <wire x1="50.8" y1="157.48" x2="50.8" y2="160.02" width="0.1524" layer="91"/>
+<pinref part="J1" gate="G$1" pin="VUSB"/>
 </segment>
 <segment>
@@
 <net name="GND" class="0">
 <segment>
-<pinref part="J1" gate="G$1" pin="GND"/>
 <wire x1="58.42" y1="147.32" x2="50.8" y2="147.32" width="0.1524" layer="91"/>
 <wire x1="50.8" y1="147.32" x2="50.8" y2="144.78" width="0.1524" layer="91"/>
 <pinref part="GND7" gate="1" pin="GND"/>
+<pinref part="J1" gate="G$1" pin="GND"/>
 </segment>
 <segment>
@@
 </segment>
 </net>
-<net name="N$42" class="0">
-<segment>
-<pinref part="U$31" gate="A" pin="D"/>
-<pinref part="J1" gate="G$1" pin="SHIELD"/>
-</segment>
-</net>
 <net name="+3V3" class="0">
 <segment>
@@
 </segment>
 </net>
-<net name="N$44" class="0">
-<segment>
-<pinref part="U$32" gate="G$1" pin="VOUT"/>
-<pinref part="U$33" gate="A" pin="D"/>
-</segment>
-</net>
 <net name="N$43" class="0">
 <segment>
@@
 </segment>
 </net>
+<net name="N$39" class="0">
+<segment>
+<pinref part="U$28" gate="A" pin="D"/>
+<pinref part="J1" gate="G$1" pin="D-"/>
+</segment>
+</net>
+<net name="N$40" class="0">
+<segment>
+<pinref part="U$29" gate="A" pin="D"/>
+<pinref part="J1" gate="G$1" pin="D+"/>
+</segment>
+</net>
+<net name="N$41" class="0">
+<segment>
+<pinref part="U$30" gate="A" pin="D"/>
+<pinref part="J1" gate="G$1" pin="ID"/>
+</segment>
+</net>
+<net name="N$42" class="0">
+<segment>
+<pinref part="U$31" gate="A" pin="D"/>
+<pinref part="J1" gate="G$1" pin="SHIELD"/>
+</segment>
+</net>
+<net name="+12V" class="0">
+<segment>
+<pinref part="U$32" gate="G$1" pin="VOUT"/>
+<wire x1="58.42" y1="93.98" x2="48.26" y2="93.98" width="0.1524" layer="91"/>
+<wire x1="48.26" y1="93.98" x2="48.26" y2="99.06" width="0.1524" layer="91"/>
+<pinref part="P+15" gate="1" pin="+12V"/>
+</segment>
+</net>

Commit message: Finished board layout, need to add mounting holes and writing
Parts:
- added R3, R4, R5, R6: (no value), rcl:R-US_0204/7
- J1: value 10118193-0001LF -> UJ2-MIBH2-4-SMT-TR; device Micro USB:10118193-0001LF -> Micro USB:UJ2-MIBH2-4-SMT-TR
Connections:
- removed net N$40 (its old number): J1.D+, U$29.D
- removed net N$41: J1.ID, U$30.D
- new net FBRAKE_PRESSURE_W/O_RES: J3.3, R1.2
- new net RBRAKE_PRESSURE_W/O_RES: J3.4, R3.1
- net +3V3: now also U$1.3V3, U$2.3V3, U2.ENABLEA
- net +5V: now also J1.1; no longer J1.VUSB
- net BACKSHIFT_LED_12V: now also R6.2; no longer R2.2
- net BACKSHIFT_LED_12V_W/O_RES: now also R6.1; no longer R2.1
- net FBRAKE_PRESSURE: now also R1.1, R2.1, U$1.34/A15, U$2.34/A15; no longer J3.3, U$1.33/A14, U$2.33/A14
- net GND: now also J1.5, R2.2, R4.1; no longer J1.GND
- net N$1: now also J1.2, U$28.D; no longer U$1.3V3
- net N$21: now also J1.3, U$29.D; no longer U$2.3V3
- net N$39: now also J1.4, U$30.D; no longer J1.D-, U$28.D
- net RBRAKE_PRESSURE: now also R3.2, R4.2, U$1.33/A14, U$2.33/A14; no longer J3.4, U$1.34/A15, U$2.34/A15
- net UPSHIFT_LED_12V: now also R5.1; no longer R1.1
- net UPSHIFT_LED_12V_W/O_RES: now also R5.2; no longer R1.2
Other:
- moved on the sheet: J1, J2, J3, J4, J5, J6, J7, R1, R2, U2

Commit message: December 2019 board finished
Parts:
- renumbered CR1 to VOLT_REG, J1 to USB, J2 to WHEEL_SPEED, J3 to BRAKE_PRESSURE, J4 to DAQ_BUTTONS_LEDS, J5 to ECVT_BUTTONS_LEDS, J6 to SPARE_ANALOG_PWM_I2C, J7 to SPARE_ANALOG_DAC, U$1 to DAQ, U$2 to ECVT, U$32 to MOTOR_DRIVER, U$57 to PENC, U$58 to SENC, U1 to DIFF_LINE_REC, U2 to LEVEL_SHIFT, XB1 to XBEE
Connections:
- net BACKSHIFT_LED renamed BKSHIFT_LED
- net BACKSHIFT_LED_12V renamed BKSHIFT_LED_12V
- net DAQ_SPARE_DAC0 renamed DAQ_SPARE_A21_DAC0
- net DAQ_SPARE_DAC1 renamed DAQ_SPARE_A22_DAC1
- net ECVT_SPARE_DAC0 renamed ECVT_SPARE_A21_DAC0
- net ECVT_SPARE_DAC1 renamed ECVT_SPARE_A22_DAC1
- net P_ENC_A renamed PENC_A
- net P_ENC_B renamed PENC_B
- net P_ENC_CHA renamed PENC_CHA
- net P_ENC_CHA/ renamed PENC_CHA/
- net P_ENC_CHB renamed PENC_CHB
- net P_ENC_CHB/ renamed PENC_CHB/
- net P_MOT_CS renamed PMOT_CS
- net P_MOT_INA renamed PMOT_INA
- net P_MOT_INB renamed PMOT_INB
- net P_MOT_PWM renamed PMOT_PWM
- net S_ENC_A renamed SENC_A
- net S_ENC_B renamed SENC_B
- net S_ENC_CHA renamed SENC_CHA
- net S_ENC_CHA/ renamed SENC_CHA/
- net S_ENC_CHB renamed SENC_CHB
- net S_ENC_CHB/ renamed SENC_CHB/
- net S_MOT_CS renamed SMOT_CS
- net S_MOT_INA renamed SMOT_INA
- net S_MOT_INB renamed SMOT_INB
- net S_MOT_PWM renamed SMOT_PWM
