File: Hardware/December 2019 Edition/EAGLE/projects/DAQ and eCVT/DAQ and eCVT.sch (EAGLE design)
At the start: 86 parts

Commit message: Minor formatting update
Parts:
- added U$1: NC, ME507:NC
Connections:
- new net N$41: LEVEL_SHIFT.NC, U$1.D
Changed lines of the file:
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@@
 <part name="R3" library="rcl" library_urn="urn:adsk.eagle:library:334" deviceset="R-US_" device="0204/7" package3d_urn="urn:adsk.eagle:package:23498/2"/>
 <part name="R4" library="rcl" library_urn="urn:adsk.eagle:library:334" deviceset="R-US_" device="0204/7" package3d_urn="urn:adsk.eagle:package:23498/2"/>
+<part name="U$1" library="ME507" deviceset="NC" device=""/>
 </parts>
 <sheets>
@@
 <attribute name="VALUE" x="41.402" y="46.99" size="1.778" layer="96" rot="R90"/>
 </instance>
+<instance part="U$1" gate="A" x="162.56" y="152.4" smashed="yes"/>
 </instances>
 <busses>
@@
 </segment>
 </net>
+<net name="N$41" class="0">
+<segment>
+<pinref part="U$1" gate="A" pin="D"/>
+<pinref part="LEVEL_SHIFT" gate="A" pin="NC"/>
+</segment>
+</net>
