File: Hardware/February 2020 Edition/EAGLE/projects/DAQ and eCVT/DAQ and eCVT.brd (EAGLE design)
At the start: 88.9 x 139.7 mm, 24 parts

Commit message: Finished schematic except RJ45 connectors and LEDs, need to redo board
Parts:
- removed DAQ, ECVT: TEENSY_3.5, Teensy:TEENSY_3.5
- removed DAQ_BUTTONS_LEDS, ECVT_BUTTONS_LEDS: TBL004-508-06BE-2GY, Screwless Terminal 6-Pole:CUI_TBL004-508-06BE-2GY
- removed MOTOR_DRIVER: POLOLU_DUAL_VNH5019, Pololo Dual VNH5019:POLOLU_DUAL_VNH5019
- removed PENC, SENC: SHF-105-01-X-D-TH, Male Header 2x5 0.05in:SHF-105-01-X-D-TH
- removed R5, R6: (no value), rcl:0204/7
- removed USB: UJ2-MIBH2-4-SMT-TR, Micro USB:CUI_UJ2-MIBH2-4-SMT-TR
- removed VOLT_REG: LD1117V33, Voltage Regulator 3.3V:TO-220
- added U$28: POLOLU_DUAL_VNH5019_BAJA, Pololo Dual VNH5019:POLOLU_DUAL_VNH5019_BAJA
- added U$31, U$33: TEENSY_3.5_BAJA, Teensy:TEENSY_3.5_BAJA
- added U1: AP2114H-3.3TRG1, Voltage Regulator 3.3V:SOT-223
- C1: value 0.1uF -> 4.7uF
- C2: value 10uF -> 4.7uF
- moved DIFF_LINE_REC 392.1 mm to (-29.2, -264.2)
- moved LEVEL_SHIFT 302.3 mm to (-50.8, -252.7)
Connections:
- net N$58 renamed ECVT_STATUS_LED_12V
- removed net BACKSHIFT_LED_12V_W/O_RES: LEVEL_SHIFT.11, R6.1
- removed net LAUNCH_CONTROL_BUTTON: ECVT_BUTTONS_LEDS.3_A, ECVT_BUTTONS_LEDS.3_B
- removed net LOGGING_STATUS_LED: LEVEL_SHIFT.3
- removed net LOGGING_STATUS_LED_12V: DAQ_BUTTONS_LEDS.5_A, DAQ_BUTTONS_LEDS.5_B, LEVEL_SHIFT.4
- removed net N$35: ECVT.35/A16
- removed net N$36: ECVT.36/A17
- removed net N$37: ECVT.37/A18
- removed net N$38: ECVT.38/A19
- removed net N$39: USB.4
- removed net N$40: USB.SH1, USB.SH2, USB.SH3, USB.SH4, USB.SH5
- removed net N$41: ECVT.4/CANRX
- removed net N$54: ECVT.VIN
- removed net N$55: DAQ.VIN
- removed net N$56: PENC.9
- removed net N$59: PENC.10
- removed net N$60: LEVEL_SHIFT.6
- removed net N$64: PENC.4
- removed net N$65: PENC.1
- removed net N$68: SENC.4
- removed net N$69: SENC.10
- removed net N$70: SENC.1
- removed net N$71: SENC.9
- removed net UPSHIFT_LED_12V_W/O_RES: LEVEL_SHIFT.13, R5.2
- new net DAQ_STATUS_LED_12V: LEVEL_SHIFT.4
- new net N$33: U$33.32/A13
- net +12V: now also U$28.VOUT; no longer DAQ_BUTTONS_LEDS.2_A, DAQ_BUTTONS_LEDS.2_B, ECVT_BUTTONS_LEDS.2_A, ECVT_BUTTONS_LEDS.2_B, MOTOR_DRIVER.VOUT
- net +3V3: now also U$28.M1EN, U$28.M2EN, U$28.VDD, U$31.3V3_LO, U$33.3V3_LO, U1.4; no longer DAQ.3V3, DAQ.3V3_LO, ECVT.3V3, ECVT.3V3_LO, MOTOR_DRIVER.3V3, MOTOR_DRIVER.M1EN, MOTOR_DRIVER.M2EN, MOTOR_DRIVER.VDD, VOLT_REG.2
- net +5V: now also U1.3; no longer DAQ_BUTTONS_LEDS.1_A, DAQ_BUTTONS_LEDS.1_B, ECVT_BUTTONS_LEDS.1_A, ECVT_BUTTONS_LEDS.1_B, MOTOR_DRIVER.5V, PENC.2, SENC.2, USB.1, VOLT_REG.3
- net BKSHIFT_LED: now also U$33.1/TX; no longer ECVT.1/TX
- net BKSHIFT_LED_12V: now also LEVEL_SHIFT.11; no longer ECVT_BUTTONS_LEDS.5_A, ECVT_BUTTONS_LEDS.5_B, R6.2
- net DAQ_ECVT\_CS: now also U$31.15/A1; no longer DAQ.15/A1
- net DAQ_ECVT\_MISO: now also U$31.12/MISO; no longer DAQ.12/MISO
- net DAQ_ECVT_CS: now also U$33.15/A1; no longer ECVT.15/A1
- net DAQ_ECVT_MISO: now also U$33.12/MISO; no longer ECVT.12/MISO
- net DAQ_ECVT_MOSI: now also U$31.11/MOSI, U$33.11/MOSI; no longer DAQ.11/MOSI, ECVT.11/MOSI
- net DAQ_ECVT_RX: now also U$31.9/CS, U$33.10/CS; no longer DAQ.9/CS, ECVT.10/CS
- net DAQ_ECVT_SCK: now also U$31.14/A0, U$33.14/A0; no longer DAQ.14/A0, ECVT.14/A0
- net DAQ_ECVT_TX: now also U$31.10/CS, U$33.9/CS; no longer DAQ.10/CS, ECVT.9/CS
- net DAQ_SPARE_A16_PWM: now also U$31.35/A16; no longer DAQ.35/A16
- net DAQ_SPARE_A17_PWM: now also U$31.36/A17; no longer DAQ.36/A17
- net DAQ_SPARE_A18_PWM_SCL: now also U$31.37/A18; no longer DAQ.37/A18
- net DAQ_SPARE_A19_PWM_SDA: now also U$31.38/A19; no longer DAQ.38/A19
- net DAQ_SPARE_A21_DAC0: now also U$31.21/DAC0; no longer DAQ.21/DAC0
- net DAQ_SPARE_A22_DAC1: now also U$31.A22/DAC1; no longer DAQ.A22/DAC1
- net DAQ_STATUS_LED: now also LEVEL_SHIFT.3, U$31.2; no longer DAQ.2
- net DAQ_XBEE_CS: now also U$31.31/A12; no longer DAQ.31/A12
- net DAQ_XBEE_MISO: now also U$31.1/TX; no longer DAQ.1/TX
- net DAQ_XBEE_MOSI: now also U$31.0/RX; no longer DAQ.0/RX
- net DAQ_XBEE_RX: now also U$31.7; no longer DAQ.7
- net DAQ_XBEE_SCK: now also U$31.32/A13; no longer DAQ.32/A13
- net DAQ_XBEE_TX: now also U$31.8; no longer DAQ.8
- net ECVT_SPARE_A21_DAC0: now also U$33.21/DAC0; no longer ECVT.21/DAC0
- net ECVT_SPARE_A22_DAC1: now also U$33.A22/DAC1; no longer ECVT.A22/DAC1
- net ECVT_STATUS_LED: now also LEVEL_SHIFT.6, U$33.2; no longer ECVT.2
- net ENGINE_SPEED: now also U$31.5, U$33.5; no longer DAQ.5, ECVT.5
- net FBRAKE_PRESSURE: now also U$31.33/A14, U$33.33/A14; no longer DAQ.33/A14, ECVT.33/A14
- net FLWHEEL_SPEED: now also U$31.29, U$33.29; no longer DAQ.29, ECVT.29
- net FRWHEEL_SPEED: now also U$31.30, U$33.30; no longer DAQ.30, ECVT.30
- net GND: now also U$28.GND, U$31.AGND, U$31.GND, U$31.GND2, U$33.AGND, U$33.GND, U$33.GND2, U1.1; no longer DAQ.AGND, DAQ.GND, DAQ.GND2, DAQ_BUTTONS_LEDS.6_A, DAQ_BUTTONS_LEDS.6_B, ECVT.AGND, ECVT.GND, ECVT.GND2, ECVT_BUTTONS_LEDS.6_A, ECVT_BUTTONS_LEDS.6_B, MOTOR_DRIVER.GND, MOTOR_DRIVER.GND1, MOTOR_DRIVER.GND2, MOTOR_DRIVER.GND3, PENC.3, SENC.3, USB.5, VOLT_REG.1
- net LAUNCH_BUTTON: now also U$33.3/CANTX; no longer ECVT.3/CANTX
- net LOGGER_BUTTON: now also U$31.3/CANTX; no longer DAQ.3/CANTX, DAQ_BUTTONS_LEDS.3_A, DAQ_BUTTONS_LEDS.3_B
- net MARKER_BUTTON: now also U$31.4/CANRX; no longer DAQ.4/CANRX, DAQ_BUTTONS_LEDS.4_A, DAQ_BUTTONS_LEDS.4_B
- net N$1: now also U1.2; no longer USB.2
- net N$10: now also U$31.22/A8; no longer DAQ.23/A9
- net N$11: now also U$31.23/A9; no longer DAQ.24
- net N$12: now also U$31.24; no longer DAQ.25
- net N$13: now also U$31.25; no longer DAQ.26
- net N$14: now also U$31.26; no longer DAQ.27
- net N$15: now also U$31.27; no longer DAQ.28
- net N$16: now also U$31.28; no longer DAQ.VUSB
- net N$17: now also U$31.39/A20; no longer DAQ.AREF
- net N$18: now also U$31.VIN; no longer DAQ.A10
- net N$19: now also U$33.3V3; no longer DAQ.A11
- net N$2: now also U$31.3V3; no longer DAQ.13/SCK
- net N$20: now also U$33.13/SCK; no longer DAQ.39/A20
- net N$21: now also LEVEL_SHIFT.12; no longer USB.3
- net N$22: now also U$33.39/A20; no longer ECVT.13/SCK
- net N$23: now also U$33.7; no longer ECVT.VUSB
- net N$24: now also U$33.8; no longer ECVT.28
- net N$25: now also U$33.28; no longer ECVT.AREF
- net N$26: now also U$33.35/A16; no longer ECVT.A10
- net N$27: now also U$33.36/A17; no longer ECVT.A11
- net N$28: now also U$33.37/A18; no longer ECVT.39/A20
- net N$29: now also U$33.38/A19; no longer ECVT.7
- net N$3: now also U$31.13/SCK; no longer DAQ.16/A2
- net N$30: now also U$33.VIN; no longer ECVT.8
- net N$31: now also U$33.4/CANRX; no longer ECVT.31/A12
- net N$32: now also U$33.31/A12; no longer ECVT.32/A13
- net N$4: now also U$31.16/A2; no longer DAQ.17/A3
- net N$5: now also U$31.17/A3; no longer DAQ.18/A4/SDA
- net N$6: now also U$31.18/A4/SDA; no longer DAQ.19/A5/SCL
- net N$7: now also U$31.19/A5/SCL; no longer DAQ.20/A6
- net N$8: now also U$31.20/A6; no longer DAQ.21/A7
- net N$9: now also U$31.21/A7; no longer DAQ.22/A8
- net PENC_A: now also U$33.24; no longer ECVT.24
- net PENC_B: now also U$33.25; no longer ECVT.25
- net PENC_CHA: no longer PENC.6
- net PENC_CHA/: no longer PENC.5
- net PENC_CHB: no longer PENC.8
- net PENC_CHB/: no longer PENC.7
- net PMOT_CS: now also U$28.M1CS, U$33.16/A2; no longer ECVT.16/A2, MOTOR_DRIVER.M1CS
- net PMOT_INA: now also U$28.M1INA, U$33.18/A4/SDA; no longer ECVT.18/A4/SDA, MOTOR_DRIVER.M1INA
- net PMOT_INB: now also U$28.M1INB, U$33.19/A5/SCL; no longer ECVT.19/A5/SCL, MOTOR_DRIVER.M1INB
- net PMOT_PWM: now also U$28.M1PWM, U$33.22/A8; no longer ECVT.22/A8, MOTOR_DRIVER.M1PWM
- net RBRAKE_PRESSURE: now also U$31.34/A15, U$33.34/A15; no longer DAQ.34/A15, ECVT.34/A15
- net RWHEELS_SPEED: now also U$31.6, U$33.6; no longer DAQ.6, ECVT.6
- net SENC_A: now also U$33.26; no longer ECVT.26
- net SENC_B: now also U$33.27; no longer ECVT.27
- net SENC_CHA: no longer SENC.6
- net SENC_CHA/: no longer SENC.5
- net SENC_CHB: no longer SENC.8
- net SENC_CHB/: no longer SENC.7
- net SMOT_CS: now also U$28.M2CS, U$33.17/A3; no longer ECVT.17/A3, MOTOR_DRIVER.M2CS
- net SMOT_INA: now also U$28.M2INA, U$33.20/A6; no longer ECVT.20/A6, MOTOR_DRIVER.M2INA
- net SMOT_INB: now also U$28.M2INB, U$33.21/A7; no longer ECVT.21/A7, MOTOR_DRIVER.M2INB
- net SMOT_PWM: now also U$28.M2PWM, U$33.23/A9; no longer ECVT.23/A9, MOTOR_DRIVER.M2PWM
- net UPSHIFT_LED: now also U$33.0/RX; no longer ECVT.0/RX
- net UPSHIFT_LED_12V: now also LEVEL_SHIFT.13; no longer ECVT_BUTTONS_LEDS.4_A, ECVT_BUTTONS_LEDS.4_B, R5.1
Routing:
- net LOGGER_BUTTON: track 148.7 -> 0.00 mm, vias 2 -> 0
- net MARKER_BUTTON: track 140.0 -> 0.00 mm, vias 2 -> 0
- net +3V3: track 276.0 -> 142.3 mm, vias 4 -> 2
- net +5V: track 108.4 -> 20.3 mm, vias 2 -> 0
- net BKSHIFT_LED: track 86.4 -> 0.00 mm
- net LAUNCH_CONTROL_BUTTON: track 77.7 -> 0.00 mm, vias 2 -> 0
- net UPSHIFT_LED: track 77.4 -> 0.00 mm
- net +12V: track 80.7 -> 7.62 mm, vias 1 -> 0
- net LOGGING_STATUS_LED: track 73.0 -> 0.00 mm
- net PENC_A: track 70.5 -> 0.00 mm, vias 4 -> 0
- net SENC_B: track 69.9 -> 0.00 mm
- net PENC_B: track 69.4 -> 0.00 mm, vias 2 -> 0
- net SENC_A: track 66.3 -> 0.00 mm
- net LOGGING_STATUS_LED_12V: track 65.5 -> 0.00 mm
- net PMOT_PWM: track 39.1 -> 0.00 mm, vias 2 -> 0
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
Commit message: Finished schematic, need to check LED wiring
Parts:
- removed SPARE_ANALOG_DAC, SPARE_ANALOG_PWM_I2C: TBL004-508-06BE-2GY, Screwless Terminal 6-Pole:CUI_TBL004-508-06BE-2GY
- added D1: LTST-C170TBKT, LED:DIOC200X125X110
- added J1, J2, J3, J4: 5558342-1, RJ45:TE_5558342-1
- added R5: (no value), rcl:R0805
- moved R2 417.4 mm to (-116.8, -326.4)
- moved R1 416.4 mm to (-127.0, -326.4), turned to 0 degrees
- moved R4 404.9 mm to (-96.5, -326.4), turned to 0 degrees
- moved R3 404.0 mm to (-106.7, -326.4)
- moved BRAKE_PRESSURE 379.7 mm to (-127.0, -287.0), turned to 0 degrees
- moved WHEEL_SPEED 367.9 mm to (-127.0, -308.6), turned to 0 degrees
Connections:
- new net N$34: D1.-, R5.1
- new net PENC_CHI: J1.1
- new net PENC_CHI/: J1.2
- new net SENC_CHI: J2.1
- new net SENC_CHI/: J2.2
- net +12V: no longer BRAKE_PRESSURE.2_A, BRAKE_PRESSURE.2_B
- net +3V3: now also BRAKE_PRESSURE.1_A, BRAKE_PRESSURE.1_B, D1.+; no longer SPARE_ANALOG_DAC.1_A, SPARE_ANALOG_DAC.1_B, SPARE_ANALOG_PWM_I2C.1_A, SPARE_ANALOG_PWM_I2C.1_B
- net +5V: now also BRAKE_PRESSURE.2_A, BRAKE_PRESSURE.2_B, J1.7, J2.7; no longer BRAKE_PRESSURE.1_A, BRAKE_PRESSURE.1_B
- net BKSHIFT_LED_12V: now also J3.3
- net DAQ_SPARE_A16_PWM: now also J4.1; no longer SPARE_ANALOG_PWM_I2C.2_A, SPARE_ANALOG_PWM_I2C.2_B
- net DAQ_SPARE_A17_PWM: now also J4.2; no longer SPARE_ANALOG_PWM_I2C.3_A, SPARE_ANALOG_PWM_I2C.3_B
- net DAQ_SPARE_A18_PWM_SCL: now also J4.3; no longer SPARE_ANALOG_PWM_I2C.4_A, SPARE_ANALOG_PWM_I2C.4_B
- net DAQ_SPARE_A19_PWM_SDA: now also J4.4; no longer SPARE_ANALOG_PWM_I2C.5_A, SPARE_ANALOG_PWM_I2C.5_B
- net DAQ_SPARE_A21_DAC0: now also J4.5; no longer SPARE_ANALOG_DAC.2_A, SPARE_ANALOG_DAC.2_B
- net DAQ_SPARE_A22_DAC1: now also J4.6; no longer SPARE_ANALOG_DAC.3_A, SPARE_ANALOG_DAC.3_B
- net DAQ_STATUS_LED_12V: now also J3.2
- net ECVT_SPARE_A21_DAC0: now also J4.7; no longer SPARE_ANALOG_DAC.4_A, SPARE_ANALOG_DAC.4_B
- net ECVT_SPARE_A22_DAC1: now also J4.8; no longer SPARE_ANALOG_DAC.5_A, SPARE_ANALOG_DAC.5_B
- net ECVT_STATUS_LED_12V: now also J3.5
- net GND: now also J1.8, J2.8, J3.8, R5.2; no longer SPARE_ANALOG_DAC.6_A, SPARE_ANALOG_DAC.6_B, SPARE_ANALOG_PWM_I2C.6_A, SPARE_ANALOG_PWM_I2C.6_B
- net LAUNCH_BUTTON: now also J3.4
- net LOGGER_BUTTON: now also J3.1
- net MARKER_BUTTON: now also J3.7
- net PENC_CHA: now also J1.3
- net PENC_CHA/: now also J1.6
- net PENC_CHB: now also J1.4
- net PENC_CHB/: now also J1.5
- net SENC_CHA: now also J2.3
- net SENC_CHA/: now also J2.6
- net SENC_CHB: now also J2.4
- net SENC_CHB/: now also J2.5
- net UPSHIFT_LED_12V: now also J3.6
Routing:
- net +3V3: track 142.3 -> 0.00 mm, vias 2 -> 0
- net FRWHEEL_SPEED: track 84.1 -> 0.00 mm, vias 1 -> 0
- net RWHEELS_SPEED: track 82.2 -> 0.00 mm
- net ECVT_SPARE_A22_DAC1: track 79.8 -> 0.00 mm, vias 2 -> 0
- net FLWHEEL_SPEED: track 77.9 -> 0.00 mm, vias 1 -> 0
- net ECVT_SPARE_A21_DAC0: track 72.6 -> 0.00 mm, vias 1 -> 0
- net ENGINE_SPEED: track 54.9 -> 0.00 mm
- net RBRAKE_PRESSURE: track 51.5 -> 0.00 mm, vias 1 -> 0
- net DAQ_SPARE_A16_PWM: track 48.5 -> 0.00 mm
- net DAQ_SPARE_A22_DAC1: track 45.8 -> 0.00 mm
- net FBRAKE_PRESSURE: track 44.3 -> 0.00 mm, vias 1 -> 0
- net DAQ_SPARE_A21_DAC0: track 41.5 -> 0.00 mm
- net DAQ_SPARE_A17_PWM: track 37.3 -> 0.00 mm
- net DAQ_SPARE_A18_PWM_SCL: track 31.2 -> 0.00 mm
- net RBRAKE_PRESSURE_W/O_RES: track 29.2 -> 0.00 mm
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