File: Hardware/February 2020 Edition/EAGLE/projects/DAQ and eCVT/DAQ and eCVT.brd (EAGLE design)
At the start: 88.9 x 114 mm, 21 parts, among them J1 5558342-1, J2 5558342-1, J3 5558342-1, J4 5558342-1, U1 AP2114H-3.3TRG1

Commit message: Wiring the board...
Parts:
- moved C1 68.0 mm to (-12.7, 82.5)
- moved U1 54.8 mm to (-12.7, 76.2)
- moved C2 44.7 mm to (-12.7, 69.8)
- moved D1 20.7 mm to (-5.08, 78.7)
- moved R5 20.7 mm to (-5.08, 74.9)
- moved R4 14.5 mm to (20.3, 74.9), turned to 180 degrees
- moved R2 14.0 mm to (20.3, 80.0)
- moved R1 2.84 mm to (7.62, 80.0), turned to 180 degrees
- moved R3 1.27 mm to (7.62, 74.9)
Routing:
- net ENGINE_SPEED: track 0.00 -> 83.3 mm, vias 0 -> 2
- net RWHEELS_SPEED: track 0.00 -> 82.8 mm, vias 0 -> 2
- net SENC_B: track 0.00 -> 63.7 mm
- net SMOT_PWM: track 0.00 -> 62.2 mm
- net SENC_A: track 0.00 -> 59.6 mm
- net SMOT_INB: track 0.00 -> 54.1 mm
- net SMOT_INA: track 0.00 -> 48.6 mm
- net PENC_B: track 0.00 -> 46.5 mm
- net PMOT_PWM: track 0.00 -> 45.4 mm
- net PENC_A: track 0.00 -> 43.2 mm
- net PMOT_INB: track 0.00 -> 35.4 mm
- net PMOT_INA: track 0.00 -> 29.9 mm
- net PENC_CHB: track 0.00 -> 22.6 mm, vias 0 -> 1
- net PENC_CHB/: track 0.00 -> 19.7 mm
- net PENC_CHA: track 0.00 -> 19.5 mm
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
Commit message: Wiring the board...
Parts:
- moved C1 58.0 mm to (38.1, 54.6)
- moved C2 51.8 mm to (38.1, 59.7)
- moved U1 48.4 mm to (31.8, 57.1)
- moved R5 17.8 mm to (12.7, 73.7)
- moved D1 12.5 mm to (6.35, 73.7)
- moved R3 7.73 mm to (6.35, 82.5)
- moved R4 7.73 mm to (19.1, 82.5)
- moved R1 1.80 mm to (6.35, 78.7)
- moved R2 1.80 mm to (19.1, 78.7)
- moved DIFF_LINE_REC 1.27 mm to (63.5, 57.8)
- moved LEVEL_SHIFT 1.27 mm to (63.5, 29.3)
Routing:
- net LOGGER_BUTTON: track 0.00 -> 110.4 mm
- net MARKER_BUTTON: track 0.00 -> 89.9 mm
- net FRWHEEL_SPEED: track 0.00 -> 84.2 mm
- net FLWHEEL_SPEED: track 0.00 -> 80.7 mm
- net LAUNCH_BUTTON: track 0.00 -> 77.0 mm
- net RBRAKE_PRESSURE_W/O_RES: track 0.00 -> 68.2 mm
- net FBRAKE_PRESSURE_W/O_RES: track 0.00 -> 58.8 mm
- net RBRAKE_PRESSURE: track 0.00 -> 38.2 mm
- net FBRAKE_PRESSURE: track 0.00 -> 36.9 mm, vias 0 -> 2
- net DAQ_ECVT_TX: track 0.00 -> 19.9 mm
- net ENGINE_SPEED: track 83.3 -> 102.1 mm
- net DAQ_ECVT_RX: track 0.00 -> 18.8 mm
- net RWHEELS_SPEED: track 82.8 -> 101.7 mm, vias 2 -> 1
- net DAQ_STATUS_LED_12V: track 0.00 -> 18.8 mm
- net ECVT_STATUS_LED_12V: track 0.00 -> 18.5 mm
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
Commit message: Wiring the board...
Connections:
- removed net DAQ_ECVT\_CS: U$31.15/A1
- net DAQ_ECVT_CS: now also U$31.15/A1
Routing:
- net DAQ_XBEE_MOSI: track 0.00 -> 72.6 mm
- net DAQ_ECVT_TX: track 19.9 -> 0.00 mm
- net DAQ_XBEE_CS: track 0.00 -> 13.8 mm
- net DAQ_XBEE_SCK: track 0.00 -> 10.7 mm
- net LOGGER_BUTTON: track 110.4 -> 100.3 mm
- net DAQ_XBEE_RX: track 0.00 -> 9.86 mm
- net DAQ_XBEE_TX: track 0.00 -> 9.09 mm
- net MARKER_BUTTON: track 89.9 -> 95.9 mm
- net DAQ_STATUS_LED: track 0.00 -> 2.15 mm, vias 0 -> 1
- net SMOT_PWM: track 62.2 -> 61.4 mm
